Commit message: backup

File: icart_mini_description/urdf/icart_mini.xacro (robot description, xacro)
@@ -7,8 +7,15 @@
   <xacro:include filename="$(find icart_mini_description)/urdf/materials.xacro" />
   <xacro:include filename="$(find icart_mini_description)/urdf/icart_mini.gazebo"/>
+  <!--Base Footprint-->
+  <link name="base_footprint" />
+  <joint name="base_joint" type="fixed">
+    <origin xyz="0 0 0" />
+    <parent link="base_footprint" />
+    <child link="base_link" />
+  </joint>
   <!-- Base Link -->
   <link name="base_link">
     <collision>
-      <origin xyz="-0.15 0 0.1" rpy="0 0 0"/>
+      <origin xyz="0.0 0.0 0.0" rpy="0 0 0"/>
       <geometry>
 	    <box size=".485 .43 .15"/>
@@ -20,8 +27,8 @@
 	    <box size=".485 .43 .15"/>
       </geometry>
-      <material name="orange"/>
+      <!-- <material name="orange"/> -->
     </visual>
     <collision name="collision">
-      <origin xyz="-0.325 0.0 0.05" rpy="0 1.5707 1.5707"/>
+      <origin xyz="0.0 0.0 0.0" rpy="0 0 0"/>
       <geometry>
         <cylinder  length="0.03" radius="0.04625"/>

File: icart_mini_description/urdf/sensors/hokuyo.urdf.xacro (robot description, xacro)
@@ -7,5 +7,5 @@
     <joint name="${name}_joint" type="fixed">
       <axis xyz="0 1 0"/>
-      <xacro:insert_block name="origin"/>
+      <insert_block name="origin"/>
       <parent link="${parent}"/>
       <child link="${name}_link"/>

File: icart_mini_description/urdf/sensors/hokuyo3d.urdf.xacro (robot description, xacro)
@@ -6,5 +6,5 @@
 	  <joint name="${name}_joint" type="fixed">
 	      <axis xyz="1 0 0"/>
-	      <xacro:insert_block name="origin"/>
+	      <insert_block name="origin"/>
 	      <parent link="${parent}"/>
 	      <child link="${name}_link"/>

File: icart_mini_description/urdf/sensors/imu.urdf.xacro (robot description, xacro)
@@ -6,5 +6,6 @@
 	  <joint name="${name}_joint" type="fixed">
 	      <axis xyz="1 0 0"/>
-	      <xacro:insert_block name="origin"/>
+	      <!--origin xyz="0 0 0.2825"/-->
+	      <insert_block name="origin"/>
 	      <parent link="${parent}"/>
 	      <child link="${name}_link"/>
@@ -35,5 +36,4 @@
             <serviceName>imu_service</serviceName>
             <gaussianNoise>0.005</gaussianNoise>
-	    <updateRate>100.0</updateRate>
         </plugin>
       </gazebo>
